File: kicad/ploterim/ploterim.kicad_sch (KiCad schematic)
At the start: 30 parts, among them SW1 nosūcējs, SW2 griezējs, U1 L78L05_TO92, U2 PC817, U3 PC817, U4 PC817

Commit message: Viss daudz glītāk
Parts:
- removed R10, R11, R15: 1k, symbol Device:R
- added J1: JACK_NOSUCEJS, Connector_Audio:Jack_3.5mm_CUI_SJ1-3523N_Horizontal, symbol Connector_Audio:AudioJack3
- added J2: JACK_LAZERS, Connector_Audio:Jack_3.5mm_CUI_SJ1-3523N_Horizontal, symbol Connector_Audio:AudioJack3
- A1: renamed from A?; value Arduino_Nano_Every -> Arduino Nano
- C1: value 1u -> 1u (neieliku); now left out of the parts list
- R10: renamed from R8; value 220 -> 100
- R11: renamed from R14; value 1K? -> 200
- R12: renamed from R13; value 220 -> 100
- R5: value 1K? -> 200
- R6: renamed from R7; value 1K? -> 200
- R7: renamed from R9; value 1K? -> 200
- R8: renamed from R6; value 220 -> 100
- R9: renamed from R12; value 1K? -> 200
- gave numbers to parts that had none: 1
Connections:
- net IND_G is gone; now on net OUT_G: A1.10 (D7), R7.1
- net IND_R is gone; now on net OUT_R: A1.8 (D5), R5.1
- net IND_Y is gone; now on net OUT_Y: A1.9 (D6), R6.1
- net VCC is gone; now on net +24V: C1.1, U1.3 (VI)
- net GND: now also J3.2 (Pin_2); no longer U2.3, U3.3, U4.3
- net OUT_G: now also R12.2; no longer U4.4
- net OUT_R: now also R8.2; no longer U2.4
- net OUT_Y: now also R10.2; no longer U3.4
- net VDD: now also A1.30 (VIN); no longer A1.27 (+5V)
- net +24V: now reaches J3.1 (Pin_1)
- net +24V: now also U2.4, U3.4, U4.4
- net OUT_GREEN: now reaches J3.4 (Pin_4)
- net OUT_GREEN: now also U4.3
- net OUT_YELLOW: now reaches J3.5 (Pin_5)
- net OUT_YELLOW: now also U3.3
- net OUT_RED: now reaches J3.6 (Pin_6)
- net OUT_RED: now also U2.3
- net LED_LAZERS: now reaches A1.13 (D10)
- net LED_LAZERS: now also R11.1
- net IND_GRIEZEJS renamed LED_NOSUCEJS
- net LED_NOSUCEJS: now also R9.1; no longer R11.1
- net IND_NOSUCEJS: no longer names the net of A1.11 (D8)
- net IND_NOSUCEJS: no longer R9.1
- net NOT_G: no longer names the net of A1.7 (D4)
- net NOT_G: no longer R12.2
- net NOT_R: no longer names the net of A1.5 (D2)
- net NOT_R: no longer R8.2
- net NOT_Y: no longer names the net of A1.6 (D3)
- net NOT_Y: no longer R10.2
- net SENSE_GRIEZEJS_A: no longer names the net of R3.2, R4.1
- net SENSE_GRIEZEJS_A: now also J2.S
- net SENSE_GRIEZEJS_B renamed IN_LAZERS
- net IN_LAZERS: now also J2.T
- net SENSE_NOSUCEJS_A: no longer names the net of R1.2, R2.1
- net SENSE_NOSUCEJS_A: now also J1.S
- net SENSE_NOSUCEJS_B renamed IN_NOSUCEJS
- net IN_NOSUCEJS: now also J1.T
- net TEST_GRIEZEJS renamed IN_TEST_LAZERS
- net TEST_NOSUCEJS renamed IN_TEST_NOSUCEJS
- no-connect marks 0 -> 21
Other:
- note added: "LEDi salikti ar 200 om rezistoriem, bet ir par spilgtu, prasītos ~1k"
- note removed: "24V ieeja"
- company: RTK CECA0 I -> RTU CECA0 I
- moved on the sheet: C1, J3

Commit message: rel3: pull-down rezistori pie optokapleriem
Parts:
- added R11, R13, R15: 100k, symbol Device:R
- renumbered R11 to R12, R12 to R14
Connections:
- net OUT_GREEN: now also R15.1
- net OUT_RED: now also R11.1
- net OUT_YELLOW: now also R13.1
- net GND renamed GNDD
- net GNDD: now also R11.2, R13.2, R15.2
